Commit message: Updated the ROS workspace

File: xembody/xembody/src/ros_ws/src/gazebo_env/description/urdf/hand.xacro (robot description, xacro)
@@ -79,4 +79,10 @@
       <mimic joint="${ns}_finger_joint1" />
     </joint>
+    <joint name="ee_joint" type="fixed">
+      <parent link="${ns}_hand"/>
+      <child link="${ns}_ee"/>
+      <origin xyz="0 0 0.096" rpy="0 0 0"/>
+    </joint>
+    <link name="${ns}_ee" />
   </xacro:macro>
 </robot>

File: xembody/xembody/src/ros_ws/src/gazebo_env/description/urdf/panda_and_panda_grippers_camera_scene_real.urdf.xacro (robot description, xacro)
@@ -1,19 +1,15 @@
 <robot name="ur5e_scene" xmlns:xacro="http://ros.org/wiki/xacro">
-  <xacro:include filename="$(find gazebo_env)/urdf/ur5_with_gripper.urdf.xacro" />
+  <xacro:include filename="$(find gazebo_env)/urdf/panda_arm_ur5e_gripper.xacro"/>
   <xacro:include filename="$(find gazebo_env)/urdf/panda_arm.xacro"/>
   <xacro:include filename="$(find gazebo_env)/urdf/hand.xacro"/>
   <link name="world" />
-  <xacro:ur5_gripper parent="world">
-      <origin xyz="0 0 10" rpy="0 0 0" />
-  </xacro:ur5_gripper>
+  <xacro:panda_with_ur5e_gripper connected_to="world" xyz="0 0 10"/>
+  <!-- We are calling this UR5 camera so we don't have to deal with stupid naming issues-->
   <xacro:include filename="$(find gazebo_env)/urdf/real_ur5_cam.urdf.xacro" />
   <xacro:sensor_d435_ur5 parent="world">
     <origin xyz="0.68760298 0.39006238 10.46098218" rpy="0.06390863  0.58797942 -2.01314893" />
   </xacro:sensor_d435_ur5>
-  <!-- Lift task-->
   <xacro:panda_arm connected_to="world" xyz="10 0 10"/>
-  <xacro:hand ns="panda" rpy="0 0 ${3 * pi/4}" connected_to="panda_link8"/>
-  <!-- Can task-->
-  <!-- <xacro:panda_arm connected_to="world" xyz="-0.56 -0.1 10.912"/>  -->
+  <xacro:hand ns="panda" rpy="0 0 ${-pi/4}" connected_to="panda_link8"/>
   <xacro:include filename="$(find gazebo_env)/urdf/real_panda_cam.urdf.xacro" />
   <xacro:sensor_d435_panda parent="world">
@@ -25,8 +21,8 @@
   </xacro:sensor_d435_panda>
   <gazebo>
-    <plugin name="ur5_and_panda_gripper_control" filename="libur5_and_panda_gripper_control_plugin.so" />
+    <plugin name="no_physics" filename="libno_physics_plugin.so" />
   </gazebo>
   <gazebo>
-    <plugin name="no_physics" filename="libno_physics_plugin.so" />
+    <plugin name="panda_and_panda_grippers_control" filename="libpanda_and_panda_grippers_control_plugin.so" />
   </gazebo>
 </robot>

File: xembody/xembody/src/ros_ws/src/gazebo_env/description/urdf/panda_arm_hand_ur5e_gripper_scene_real.urdf.xacro (robot description, xacro)
@@ -4,5 +4,5 @@
   <link name="world" />
   <!-- Lift task-->
-  <xacro:panda_arm connected_to="world" xyz="0 0 0"/>
+  <xacro:panda_with_ur5e_gripper connected_to="world" xyz="0 0 0"/>
   <gazebo>
     <plugin name="no_physics" filename="libno_physics_plugin.so" />

File: xembody/xembody/src/ros_ws/src/gazebo_env/description/urdf/panda_arm_ur5e_gripper.xacro (robot description, xacro)
@@ -1,6 +1,6 @@
 <?xml version='1.0' encoding='utf-8'?>
 <robot xmlns:xacro="http://www.ros.org/wiki/xacro" name="panda">
-  <xacro:macro name="panda_arm"
-    params="arm_id:='panda' description_pkg:='franka_description' connected_to:='' xyz:='0 0 0' rpy:='0 0 0'">
+  <xacro:macro name="panda_with_ur5e_gripper"
+    params="arm_id:='panda_with_ur5_gripper' description_pkg:='franka_description' connected_to:='' xyz:='0 0 0' rpy:='0 0 0'">
     <xacro:unless value="${not connected_to}">
       <joint name="${arm_id}_joint_${connected_to}" type="fixed">
@@ -294,4 +294,10 @@
       </inertial>
     </link>
+    <joint name="ur5_ee_gripper_joint" type="fixed">
+      <parent link="robotiq_85_base_link" />
+      <child link="ur5_ee_gripper" />
+      <origin rpy="-1.571 0 -1.571" xyz="0.127 0.0 0.0" />
+    </joint>
+    <link name="ur5_ee_gripper" />
     <joint name="robotiq_85_left_knuckle_joint" type="revolute">
       <parent link="robotiq_85_base_link" />

File: xembody/xembody/src/ros_ws/src/gazebo_env/description/urdf/panda_ur5_gripper_ik_real.urdf (robot description, URDF)
Before this commit: robot panda, 23 links, 22 joints
Links:
- removed link panda_link0
- removed link panda_link1
- removed link panda_link2
- removed link panda_link3
- removed link panda_link4
- removed link panda_link5
- removed link panda_link6
- removed link panda_link7
- removed link panda_link8
- added link panda_with_ur5_gripper_link0, mass 2.8142028896; collision mesh filename=file:///home/lawrence/xembody/cross_embodiment_ws/install/g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; visual mesh filename=file:///home/lawrence/xembody/cross_embodiment_ws/install/g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
- added link panda_with_ur5_gripper_link1, mass 2.3599995791; collision mesh filename=file:///home/lawrence/xembody/cross_embodiment_ws/install/g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; visual mesh filename=file:///home/lawrence/xembody/cross_embodiment_ws/install/g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
- added link panda_with_ur5_gripper_link2, mass 2.379518833; collision mesh filename=file:///home/lawrence/xembody/cross_embodiment_ws/install/g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; visual mesh filename=file:///home/lawrence/xembody/cross_embodiment_ws/install/g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
- added link panda_with_ur5_gripper_link3, mass 2.6498823337; collision mesh filename=file:///home/lawrence/xembody/cross_embodiment_ws/install/g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; visual mesh filename=file:///home/lawrence/xembody/cross_embodiment_ws/install/g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
- added link panda_with_ur5_gripper_link4, mass 2.6948018744; collision mesh filename=file:///home/lawrence/xembody/cross_embodiment_ws/install/g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; visual mesh filename=file:///home/lawrence/xembody/cross_embodiment_ws/install/g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
- added link panda_with_ur5_gripper_link5, mass 2.9812816864; collision mesh filename=file:///home/lawrence/xembody/cross_embodiment_ws/install/g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; visual mesh filename=file:///home/lawrence/xembody/cross_embodiment_ws/install/g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
- added link panda_with_ur5_gripper_link6, mass 1.1285806309; collision mesh filename=file:///home/lawrence/xembody/cross_embodiment_ws/install/g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; visual mesh filename=file:///home/lawrence/xembody/cross_embodiment_ws/install/g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
- added link panda_with_ur5_gripper_link7, mass 0.4052912465; collision mesh filename=file:///home/lawrence/xembody/cross_embodiment_ws/install/g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; visual mesh filename=file:///home/lawrence/xembody/cross_embodiment_ws/install/g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
- added link panda_with_ur5_gripper_link8
- added link ur5_ee_gripper
- link robotiq_85_base_link: geometry collision mesh filename=file:///home/lawrence/xembody/cross_embodiment_ws/install/g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; visual mesh filename=file:///home/lawrence/xembody/cross_embodiment_ws/install/g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
- link robotiq_85_left_finger_link: geometry collision mesh filename=file:///home/lawrence/xembody/cross_embodiment_ws/install/g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; visual mesh filename=file:///home/lawrence/xembody/cross_embodiment_ws/install/g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
- link robotiq_85_left_finger_tip_link: geometry collision mesh filename=file:///home/lawrence/xembody/cross_embodiment_ws/install/g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; visual mesh filename=file:///home/lawrence/xembody/cross_embodiment_ws/install/g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
- link robotiq_85_left_inner_knuckle_link: geometry collision mesh filename=file:///home/lawrence/xembody/cross_embodiment_ws/install/g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; visual mesh filename=file:///home/lawrence/xembody/cross_embodiment_ws/install/g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
- link robotiq_85_left_knuckle_link: geometry collision mesh filename=file:///home/lawrence/xembody/cross_embodiment_ws/install/g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; visual mesh filename=file:///home/lawrence/xembody/cross_embodiment_ws/install/g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
- link robotiq_85_right_finger_link: geometry collision mesh filename=file:///home/lawrence/xembody/cross_embodiment_ws/install/g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; visual mesh filename=file:///home/lawrence/xembody/cross_embodiment_ws/install/g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
- link robotiq_85_right_finger_tip_link: geometry collision mesh filename=file:///home/lawrence/xembody/cross_embodiment_ws/install/g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; visual mesh filename=file:///home/lawrence/xembody/cross_embodiment_ws/install/g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
- link robotiq_85_right_inner_knuckle_link: geometry collision mesh filename=file:///home/lawrence/xembody/cross_embodiment_ws/install/g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; visual mesh filename=file:///home/lawrence/xembody/cross_embodiment_ws/install/g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
- link robotiq_85_right_knuckle_link: geometry collision mesh filename=file:///home/lawrence/xembody/cross_embodiment_ws/install/g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; visual mesh filename=file:///home/lawrence/xembody/cross_embodiment_ws/install/g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
Joints:
- removed joint panda_joint1
- removed joint panda_joint2
- removed joint panda_joint3
- removed joint panda_joint4
- removed joint panda_joint5
- removed joint panda_joint6
- removed joint panda_joint7
- removed joint panda_joint8
- removed joint panda_joint_world
- added joint panda_with_ur5_gripper_joint1: type revolute, parent panda_with_ur5_gripper_link0, child panda_with_ur5_gripper_link1, origin xyz=0 0 0.333 rpy=0 0 0, axis 0 0 1, limit lower=-2.8973 upper=2.8973 effort=87 velocity=2.1750
- added joint panda_with_ur5_gripper_joint2: type revolute, parent panda_with_ur5_gripper_link1, child panda_with_ur5_gripper_link2, origin xyz=0 0 0 rpy=-1.5707963267948966 0 0, axis 0 0 1, limit lower=-1.7628 upper=1.7628 effort=87 velocity=2.1750
- added joint panda_with_ur5_gripper_joint3: type revolute, parent panda_with_ur5_gripper_link2, child panda_with_ur5_gripper_link3, origin xyz=0 -0.316 0 rpy=1.5707963267948966 0 0, axis 0 0 1, limit lower=-2.8973 upper=2.8973 effort=87 velocity=2.1750
- added joint panda_with_ur5_gripper_joint4: type revolute, parent panda_with_ur5_gripper_link3, child panda_with_ur5_gripper_link4, origin xyz=0.0825 0 0 rpy=1.5707963267948966 0 0, axis 0 0 1, limit lower=-3.0718 upper=-0.0698 effort=87 velocity=2.1750
- added joint panda_with_ur5_gripper_joint5: type revolute, parent panda_with_ur5_gripper_link4, child panda_with_ur5_gripper_link5, origin xyz=-0.0825 0.384 0 rpy=-1.5707963267948966 0 0, axis 0 0 1, limit lower=-2.8973 upper=2.8973 effort=12 velocity=2.6100
- added joint panda_with_ur5_gripper_joint6: type revolute, parent panda_with_ur5_gripper_link5, child panda_with_ur5_gripper_link6, origin xyz=0 0 0 rpy=1.5707963267948966 0 0, axis 0 0 1, limit lower=-0.0175 upper=3.7525 effort=12 velocity=2.6100
- added joint panda_with_ur5_gripper_joint7: type revolute, parent panda_with_ur5_gripper_link6, child panda_with_ur5_gripper_link7, origin xyz=0.088 0 0 rpy=1.5707963267948966 0 0, axis 0 0 1, limit lower=-2.8973 upper=2.8973 effort=12 velocity=2.6100
- added joint panda_with_ur5_gripper_joint8: type fixed, parent panda_with_ur5_gripper_link7, child panda_with_ur5_gripper_link8, origin xyz=0 0 0.107 rpy=0 0 0, axis 0 0 0
- added joint panda_with_ur5_gripper_joint_world: type fixed, parent world, child panda_with_ur5_gripper_link0, origin xyz=0 0 0 rpy=0 0 0
- added joint ur5_ee_gripper_joint: type fixed, parent robotiq_85_base_link, child ur5_ee_gripper, origin xyz=0.127 0.0 0.0 rpy=-1.571 0 -1.571
- joint arm_gripper_adapter_joint: parent panda_link8 -> panda_with_ur5_gripper_link8
- joint ee_fixed_joint: parent panda_link8 -> panda_with_ur5_gripper_link8
- joint link8_to_panda_ee_link_fixed_joint: parent panda_link8 -> panda_with_ur5_gripper_link8
- joint wrist_3_link-tool0_fixed_joint: parent panda_link8 -> panda_with_ur5_gripper_link8

File: xembody/xembody/src/ros_ws/src/gazebo_env/description/urdf/ur5_ik_real.urdf (robot description, URDF)
Before this commit: robot ur5e_scene, 23 links, 22 joints
Links:
- added link ur5_ee_gripper
Joints:
- added joint tool0-ur5_ee_gripper: type fixed, parent tool0, child ur5_ee_gripper, origin xyz=0 0 0.143 rpy=0 0 0

File: xembody/xembody/src/ros_ws/src/gazebo_env/description/urdf/ur5_with_gripper.urdf.xacro (robot description, xacro)
@@ -263,4 +263,10 @@
       <child link="tool0" />
     </joint>
+    <joint name="tool0-ur5_ee_gripper" type="fixed">
+      <origin rpy="0 0 0" xyz="0 0 0.143" />
+      <parent link="tool0" />
+      <child link="ur5_ee_gripper" />
+    </joint>
+    <link name="ur5_ee_gripper" />
     <!-- <joint name="arm_gripper_joint" type="fixed">
       <parent link="wrist_3_link" />

File: xembody/xembody/src/ros_ws/src/gazebo_env/description/urdf/ur5_with_gripper_camera_scene_real.urdf.xacro (robot description, xacro)
@@ -2,10 +2,16 @@
   <xacro:include filename="$(find gazebo_env)/urdf/ur5_with_gripper.urdf.xacro" />
   <link name="world" />
-  <xacro:ur5e_gripper parent="world">
+  <xacro:ur5_gripper parent="world">
       <origin xyz="0 0 10" rpy="0 0 0" />
-  </xacro:ur5e_gripper>
+  </xacro:ur5_gripper>
   <xacro:include filename="$(find gazebo_env)/urdf/real_ur5_cam.urdf.xacro" />
   <xacro:sensor_d435_ur5 parent="world">
     <origin xyz="0.90641516 -0.08090482 10.6424972" rpy="0.0588804 0.6888795 3.1219407" />
   </xacro:sensor_d435_ur5>
+  <gazebo>
+    <plugin name="no_physics" filename="libno_physics_plugin.so" />
+  </gazebo>
+  <gazebo>
+    <plugin name="ur5_control" filename="libur5e_control_plugin.so" />
+  </gazebo>
 </robot>
