Commit message: Updated with inpaint code

File: xembody/xembody/src/ros_ws/src/gazebo_env/description/urdf/d435.urdf.xacro (robot description, xacro)
@@ -109,6 +109,6 @@
             <image>
                 <format>R8G8B8</format>
-                <width>256</width>
-                <height>256</height>
+                <width>512</width>
+                <height>512</height>
                 <!-- <width>256</width>
                 <height>256</height> -->

File: xembody/xembody/src/ros_ws/src/gazebo_env/description/urdf/panda_arm_hand_camera_scene_robosuite_can.urdf.xacro (robot description, xacro)
@@ -13,5 +13,5 @@
     <!-- for some reason we have to modify the xyz because it is a little shifted-->
     <!-- Lift task-->
-    <origin xyz="0.516 0.018 11.749" rpy="0 0.7840421 3.1415927" />
+    <origin xyz="1.016 0.018 11.749" rpy="0 0.7840421 3.1415927" />
     <!-- Can task-->
     <!-- <origin xyz="1.016 0.018 11.749" rpy="0 0.7840421 3.1415927" />  -->
