Commit message: Try to finish cleanup

File: xembody/xembody/src/ros_ws/src/gazebo_env/description/urdf/real_panda_cam.urdf.xacro (robot description, xacro)
@@ -25,12 +25,4 @@
     </joint>
     <link name="panda_camera_link">
-      <visual>
-        <!-- the mesh origin is at front plate in between the two infrared camera axes -->
-        <origin rpy="1.5707963267948966 0 1.5707963267948966" xyz="0.0043 -0.0175 0" />
-        <geometry>
-          <mesh
-            filename="file://$(find gazebo_env)/meshes/d435/d435.dae" />
-        </geometry>
-      </visual>
       <collision>
         <origin rpy="0 0 0" xyz="0 -0.0175 0" />

File: xembody/xembody/src/ros_ws/src/gazebo_env/description/urdf/real_panda_cam_left.urdf.xacro (robot description, xacro)
@@ -25,12 +25,4 @@
     </joint>
     <link name="panda_left_camera_link">
-      <visual>
-        <!-- the mesh origin is at front plate in between the two infrared camera axes -->
-        <origin rpy="1.5707963267948966 0 1.5707963267948966" xyz="0.0043 -0.0175 0" />
-        <geometry>
-          <mesh
-            filename="file://$(find gazebo_env)/meshes/d435/d435.dae" />
-        </geometry>
-      </visual>
       <collision>
         <origin rpy="0 0 0" xyz="0 -0.0175 0" />

File: xembody/xembody/src/ros_ws/src/gazebo_env/description/urdf/real_panda_cam_no_gripper.urdf.xacro (robot description, xacro)
@@ -25,12 +25,4 @@
     </joint>
     <link name="panda_no_gripper_camera_link">
-      <visual>
-        <!-- the mesh origin is at front plate in between the two infrared camera axes -->
-        <origin rpy="1.5707963267948966 0 1.5707963267948966" xyz="0.0043 -0.0175 0" />
-        <geometry>
-          <mesh
-            filename="file://$(find gazebo_env)/meshes/d435/d435.dae" />
-        </geometry>
-      </visual>
       <collision>
         <origin rpy="0 0 0" xyz="0 -0.0175 0" />

File: xembody/xembody/src/ros_ws/src/gazebo_env/description/urdf/real_panda_cam_right.urdf.xacro (robot description, xacro)
@@ -25,12 +25,4 @@
     </joint>
     <link name="panda_right_camera_link">
-      <visual>
-        <!-- the mesh origin is at front plate in between the two infrared camera axes -->
-        <origin rpy="1.5707963267948966 0 1.5707963267948966" xyz="0.0043 -0.0175 0" />
-        <geometry>
-          <mesh
-            filename="file://$(find gazebo_env)/meshes/d435/d435.dae" />
-        </geometry>
-      </visual>
       <collision>
         <origin rpy="0 0 0" xyz="0 -0.0175 0" />

File: xembody/xembody/src/ros_ws/src/gazebo_env/description/urdf/real_ur5_cam.urdf.xacro (robot description, xacro)
@@ -25,12 +25,4 @@
     </joint>
     <link name="ur5_camera_link">
-      <visual>
-        <!-- the mesh origin is at front plate in between the two infrared camera axes -->
-        <origin rpy="1.5707963267948966 0 1.5707963267948966" xyz="0.0043 -0.0175 0" />
-        <geometry>
-          <mesh
-            filename="file://$(find gazebo_env)/meshes/d435/d435.dae" />
-        </geometry>
-      </visual>
       <collision>
         <origin rpy="0 0 0" xyz="0 -0.0175 0" />

File: xembody/xembody/src/ros_ws/src/gazebo_env/description/urdf/real_ur5_cam_left.urdf.xacro (robot description, xacro)
@@ -25,12 +25,4 @@
     </joint>
     <link name="ur5_left_camera_link">
-      <visual>
-        <!-- the mesh origin is at front plate in between the two infrared camera axes -->
-        <origin rpy="1.5707963267948966 0 1.5707963267948966" xyz="0.0043 -0.0175 0" />
-        <geometry>
-          <mesh
-            filename="file://$(find gazebo_env)/meshes/d435/d435.dae" />
-        </geometry>
-      </visual>
       <collision>
         <origin rpy="0 0 0" xyz="0 -0.0175 0" />

File: xembody/xembody/src/ros_ws/src/gazebo_env/description/urdf/real_ur5_cam_right.urdf.xacro (robot description, xacro)
@@ -25,12 +25,4 @@
     </joint>
     <link name="ur5_right_camera_link">
-      <visual>
-        <!-- the mesh origin is at front plate in between the two infrared camera axes -->
-        <origin rpy="1.5707963267948966 0 1.5707963267948966" xyz="0.0043 -0.0175 0" />
-        <geometry>
-          <mesh
-            filename="file://$(find gazebo_env)/meshes/d435/d435.dae" />
-        </geometry>
-      </visual>
       <collision>
         <origin rpy="0 0 0" xyz="0 -0.0175 0" />
