Commit message: Starting gazebo cleanup

File: xembody/xembody/src/ros_ws/src/gazebo_env/description/urdf/real_ur5_cam_right_wrist.urdf.xacro (robot description, xacro)
@@ -5,26 +5,25 @@
 <!-- =================================================================================== -->
 <robot name="realsense2_camera" xmlns:xacro="http://ros.org/wiki/xacro">
-  <xacro:macro name="sensor_d435_ur5_left"
+  <xacro:macro name="sensor_d435_ur5_right_wrist"
     params="parent *origin name:=camera use_nominal_extrinsics:=false add_plug:=false use_mesh:=true">
-    <material name="ur5_left_aluminum">
+    <material name="ur5_right_aluminum">
       <color rgba="0.5 0.5 0.5 1" />
     </material>
-    <material name="ur5_left_plastic">
+    <material name="ur5_right_plastic">
       <color rgba="0.1 0.1 0.1 1" />
     </material>
-    <joint name="ur5_left_camera_joint" type="fixed">
+    <joint name="ur5_right_camera_joint" type="fixed">
       <xacro:insert_block name="origin" />
       <parent link="${parent}" />
-      <child link="ur5_left_camera_bottom_screw_frame" />
+      <child link="ur5_right_camera_bottom_screw_frame" />
     </joint>
-    <link name="ur5_left_camera_bottom_screw_frame" />
-    <joint name="ur5_left_camera_link_joint" type="fixed">
+    <link name="ur5_right_camera_bottom_screw_frame" />
+    <joint name="ur5_right_camera_link_joint" type="fixed">
       <origin rpy="0 0 0" xyz="0.010600000000000002 0.0175 0.0125" />
-      <parent link="ur5_left_camera_bottom_screw_frame" />
-      <child link="ur5_left_camera_link" />
+      <parent link="ur5_right_camera_bottom_screw_frame" />
+      <child link="ur5_right_camera_link" />
     </joint>
-    <link name="ur5_left_camera_link">
-      <visual>
-        <!-- the mesh origin is at front plate in between the two infrared camera axes -->
+    <link name="ur5_right_camera_link">
+      <!-- <visual>
         <origin rpy="1.5707963267948966 0 1.5707963267948966" xyz="0.0043 -0.0175 0" />
         <geometry>
@@ -32,5 +31,5 @@
             filename="file://$(find gazebo_env)/meshes/d435/d435.dae" />
         </geometry>
-      </visual>
+      </visual> -->
       <collision>
         <origin rpy="0 0 0" xyz="0 -0.0175 0" />
@@ -47,64 +46,65 @@
     </link>
     <!-- camera depth joints and links -->
-    <joint name="ur5_left_camera_depth_joint" type="fixed">
+    <joint name="ur5_right_camera_depth_joint" type="fixed">
       <origin rpy="0 0 0" xyz="0 0 0" />
-      <parent link="ur5_left_camera_link" />
-      <child link="ur5_left_camera_depth_frame" />
+      <parent link="ur5_right_camera_link" />
+      <child link="ur5_right_camera_depth_frame" />
     </joint>
-    <link name="ur5_left_camera_depth_frame" />
-    <joint name="ur5_left_camera_depth_optical_joint" type="fixed">
+    <link name="ur5_right_camera_depth_frame" />
+    <joint name="ur5_right_camera_depth_optical_joint" type="fixed">
       <origin rpy="-1.5707963267948966 0 -1.5707963267948966" xyz="0 0 0" />
-      <parent link="ur5_left_camera_depth_frame" />
-      <child link="ur5_left_camera_depth_optical_frame" />
+      <parent link="ur5_right_camera_depth_frame" />
+      <child link="ur5_right_camera_depth_optical_frame" />
     </joint>
-    <link name="ur5_left_camera_depth_optical_frame" />
-    <!-- camera left IR joints and links -->
-    <joint name="ur5_left_camera_infra1_joint" type="fixed">
+    <link name="ur5_right_camera_depth_optical_frame" />
+    <!-- camera right IR joints and links -->
+    <joint name="ur5_right_camera_infra1_joint" type="fixed">
       <origin rpy="0 0 0" xyz="0 0.0 0" />
-      <parent link="ur5_left_camera_link" />
-      <child link="ur5_left_camera_infra1_frame" />
+      <parent link="ur5_right_camera_link" />
+      <child link="ur5_right_camera_infra1_frame" />
     </joint>
-    <link name="ur5_left_camera_infra1_frame" />
-    <joint name="ur5_left_camera_infra1_optical_joint" type="fixed">
+    <link name="ur5_right_camera_infra1_frame" />
+    <joint name="ur5_right_camera_infra1_optical_joint" type="fixed">
       <origin rpy="-1.5707963267948966 0 -1.5707963267948966" xyz="0 0 0" />
-      <parent link="ur5_left_camera_infra1_frame" />
-      <child link="ur5_left_camera_infra1_optical_frame" />
+      <parent link="ur5_right_camera_infra1_frame" />
+      <child link="ur5_right_camera_infra1_optical_frame" />
     </joint>
-    <link name="ur5_left_camera_infra1_optical_frame" />
+    <link name="ur5_right_camera_infra1_optical_frame" />
     <!-- camera right IR joints and links -->
-    <joint name="ur5_left_camera_infra2_joint" type="fixed">
+    <joint name="ur5_right_camera_infra2_joint" type="fixed">
       <origin rpy="0 0 0" xyz="0 -0.05 0" />
-      <parent link="ur5_left_camera_link" />
-      <child link="ur5_left_camera_infra2_frame" />
+      <parent link="ur5_right_camera_link" />
+      <child link="ur5_right_camera_infra2_frame" />
     </joint>
-    <link name="ur5_left_camera_infra2_frame" />
-    <joint name="ur5_left_camera_infra2_optical_joint" type="fixed">
+    <link name="ur5_right_camera_infra2_frame" />
+    <joint name="ur5_right_camera_infra2_optical_joint" type="fixed">
       <origin rpy="-1.5707963267948966 0 -1.5707963267948966" xyz="0 0 0" />
-      <parent link="ur5_left_camera_infra2_frame" />
-      <child link="ur5_left_camera_infra2_optical_frame" />
+      <parent link="ur5_right_camera_infra2_frame" />
+      <child link="ur5_right_camera_infra2_optical_frame" />
     </joint>
-    <link name="ur5_left_camera_infra2_optical_frame" />
+    <link name="ur5_right_camera_infra2_optical_frame" />
     <!-- camera color joints and links -->
-    <joint name="ur5_left_camera_color_joint" type="fixed">
+    <joint name="ur5_right_camera_color_joint" type="fixed">
       <origin rpy="0 0 0" xyz="0 0.015 0" />
-      <parent link="ur5_left_camera_link" />
-      <child link="ur5_left_camera_color_frame" />
+      <parent link="ur5_right_camera_link" />
+      <child link="ur5_right_camera_color_frame" />
     </joint>
-    <link name="ur5_left_camera_color_frame" />
-    <joint name="ur5_left_camera_color_optical_joint" type="fixed">
+    <link name="ur5_right_camera_color_frame" />
+    <joint name="ur5_right_camera_color_optical_joint" type="fixed">
       <origin rpy="-1.5707963267948966 0 -1.5707963267948966" xyz="0 0 0" />
-      <parent link="ur5_left_camera_color_frame" />
-      <child link="ur5_left_camera_color_optical_frame" />
+      <parent link="ur5_right_camera_color_frame" />
+      <child link="ur5_right_camera_color_optical_frame" />
     </joint>
-    <link name="ur5_left_camera_color_optical_frame" />
-    <gazebo reference="ur5_left_camera_link">
+    <link name="ur5_right_camera_color_optical_frame" />
+    <gazebo reference="ur5_right_camera_link">
       <material>Gazebo/TurquoiseGlowOutline </material>
-      <sensor name="ur5_left_camera" type="depth">
+      <sensor name="ur5_right_camera" type="depth">
         <pose> 0 0 0 0 0 0 </pose>
         <visualize>false</visualize>
         <update_rate>30</update_rate>
         <!-- Focal Length = Width * 0.5 / tan(Hor. FOV (in radians) * 0.5)-->
+        <!-- Hor. FOV (in radians) = 2 *arctan(Width * 0.5 / Focal Length)-->
         <camera>
-            <horizontal_fov>1.769165872</horizontal_fov>
+            <horizontal_fov>1.768165077</horizontal_fov>
             <image>
                 <format>R8G8B8</format>
@@ -119,6 +119,6 @@
             </clip>
         </camera>
-        <plugin name="ur5_left_camera_controller" filename="libgazebo_ros_camera.so">
-            <frame_name>ur5_left_camera_color_optical_frame</frame_name>
+        <plugin name="ur5_right_camera_controller" filename="libgazebo_ros_camera.so">
+            <frame_name>ur5_right_camera_color_optical_frame</frame_name>
             <!-- <cx>647.53735352</cx> -->
             <!-- <cy>367.65203857</cy> -->

File: xembody/xembody/src/ros_ws/src/gazebo_env/description/urdf/ur5_and_panda_gripper_multi_camera_early_inpaint_scene_real.urdf.xacro (robot description, xacro)
@@ -10,8 +10,8 @@
   <xacro:include filename="$(find gazebo_env)/urdf/real_ur5_cam_right.urdf.xacro" />
   <xacro:sensor_d435_ur5_left parent="world">
-    <origin xyz="0.676 0.401 10.455" rpy="0.0994744   0.60025461 -2.00644895" />
+    <origin xyz="0.65147084 0.41435814 10.51452678" rpy="0.11023138  0.57410099 -1.9646524" />
   </xacro:sensor_d435_ur5_left>
   <xacro:sensor_d435_ur5_right parent="world">
-    <origin xyz="0.832 -0.03 10.410" rpy="3.10103845 0.95510487 3.08504758" />
+    <origin xyz="0.5538436 0.47336682 10.50176154" rpy="0.05888073  0.52934421 -1.97405572" />
   </xacro:sensor_d435_ur5_right>
   <!-- Lift task-->
@@ -23,8 +23,8 @@
   <xacro:include filename="$(find gazebo_env)/urdf/real_panda_cam_right.urdf.xacro" />
   <xacro:sensor_d435_panda_left parent="world">
-    <origin xyz="10.676 0.401 10.455" rpy="0.0994744   0.60025461 -2.00644895"/>
+    <origin xyz="10.65147084 0.41435814 10.51452678" rpy="0.11023138  0.57410099 -1.9646524" />
   </xacro:sensor_d435_panda_left>
   <xacro:sensor_d435_panda_right parent="world">
-    <origin xyz="10.832 -0.03 10.410" rpy="3.10103845 0.95510487 3.08504758" />
+    <origin xyz="10.5538436 0.47336682 10.50176154" rpy="0.05888073  0.52934421 -1.97405572" />
   </xacro:sensor_d435_panda_right>
   <xacro:include filename="$(find gazebo_env)/urdf/ur5_with_no_gripper.urdf.xacro" />
@@ -34,9 +34,9 @@
   <xacro:include filename="$(find gazebo_env)/urdf/real_ur5_cam_no_gripper_left.urdf.xacro" />
   <xacro:sensor_d435_ur5_no_gripper_left parent="world">
-    <origin xyz="10.676 20.401 10.455" rpy="0.0994744   0.60025461 -2.00644895" />
+    <origin xyz="10.68760298 20.39006238 10.46098218" rpy="0.06390863  0.58797942 -2.01314893" />
   </xacro:sensor_d435_ur5_no_gripper_left>
   <xacro:include filename="$(find gazebo_env)/urdf/real_ur5_cam_no_gripper_right.urdf.xacro" />
   <xacro:sensor_d435_ur5_no_gripper_right parent="world">
-    <origin xyz="10.832 19.97 10.410" rpy="3.10103845 0.95510487 3.08504758" />
+    <origin xyz="10.68760298 25.39006238 10.46098218" rpy="0.06390863  0.58797942 -2.01314893" />
   </xacro:sensor_d435_ur5_no_gripper_right>
   <gazebo>
