Commit message: Updated luminances

File: mirage/mirage/ros_ws/src/gazebo_env/description/urdf/panda_arm_hand_camera_scene_robosuite_can.urdf.xacro (robot description, xacro)
@@ -9,12 +9,12 @@
   <!-- <xacro:panda_arm connected_to="world" xyz="-0.56 -0.1 10.912"/>  -->
   <xacro:hand ns="panda" rpy="0 0 ${-pi/4}" connected_to="panda_link8"/>
-  <xacro:include filename="$(find gazebo_env)/urdf/d435.urdf.xacro" />
-  <xacro:sensor_d435 parent="world">
+  <xacro:include filename="$(find gazebo_env)/urdf/d435_robosuite.urdf.xacro" />
+  <xacro:sensor_d435_robosuite parent="world">
     <!-- for some reason we have to modify the xyz because it is a little shifted-->
     <!-- Lift task-->
-    <origin xyz="0.516 0.018 11.749" rpy="0 0.7840421 3.1415927" />
+    <origin xyz="1.016 0.018 11.749" rpy="0 0.7840421 3.1415927" />
     <!-- Can task-->
     <!-- <origin xyz="1.016 0.018 11.749" rpy="0 0.7840421 3.1415927" />  -->
-  </xacro:sensor_d435>
+  </xacro:sensor_d435_robosuite>
   <gazebo>
     <plugin name="no_physics" filename="libno_physics_plugin.so" />

File: mirage/mirage/ros_ws/src/gazebo_env/description/urdf/panda_arm_hand_camera_scene_robosuite_lift_square_stack_three_threading.urdf.xacro (robot description, xacro)
@@ -9,6 +9,6 @@
   <!-- <xacro:panda_arm connected_to="world" xyz="-0.56 -0.1 10.912"/>  -->
   <xacro:hand ns="panda" rpy="0 0 ${-pi/4}" connected_to="panda_link8"/>
-  <xacro:include filename="$(find gazebo_env)/urdf/d435.urdf.xacro" />
-  <xacro:sensor_d435 parent="world">
+  <xacro:include filename="$(find gazebo_env)/urdf/d435_robosuite.urdf.xacro" />
+  <xacro:sensor_d435_robosuite parent="world">
     <!-- for some reason we have to modify the xyz because it is a little shifted-->
     <!-- Lift task-->
@@ -16,5 +16,5 @@
     <!-- Can task-->
     <!-- <origin xyz="1.016 0.018 11.749" rpy="0 0.7840421 3.1415927" />  -->
-  </xacro:sensor_d435>
+  </xacro:sensor_d435_robosuite>
   <gazebo>
     <plugin name="no_physics" filename="libno_physics_plugin.so" />

File: mirage/mirage/ros_ws/src/gazebo_env/description/urdf/panda_arm_hand_camera_scene_robosuite_three_piece_assembly.urdf.xacro (robot description, xacro)
@@ -9,6 +9,6 @@
   <!-- <xacro:panda_arm connected_to="world" xyz="-0.56 -0.1 10.912"/>  -->
   <xacro:hand ns="panda" rpy="0 0 ${-pi/4}" connected_to="panda_link8"/>
-  <xacro:include filename="$(find gazebo_env)/urdf/d435.urdf.xacro" />
-  <xacro:sensor_d435 parent="world">
+  <xacro:include filename="$(find gazebo_env)/urdf/d435_robosuite.urdf.xacro" />
+  <xacro:sensor_d435_robosuite parent="world">
     <!-- for some reason we have to modify the xyz because it is a little shifted-->
     <!-- Lift task-->
@@ -16,5 +16,5 @@
     <!-- Can task-->
     <!-- <origin xyz="1.016 0.018 11.749" rpy="0 0.7840421 3.1415927" />  -->
-  </xacro:sensor_d435>
+  </xacro:sensor_d435_robosuite>
   <gazebo>
     <plugin name="no_physics" filename="libno_physics_plugin.so" />
